File: circuit/boards and schematics/20220806/main.brd (EAGLE design)
At the start: 70 x 30 mm, 9 parts, among them U1 ESP32-DEVKITC-32D, X1 JST-XH-05-PIN-LONG-PAD

Commit message: created garber files
Routing:
- net GND: track 111.6 -> 152.2 mm
Changed lines of the file:
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@@
 <wire x1="9.25" y1="9.75" x2="9" y2="9.92" width="0.762" layer="16"/>
 <wire x1="41.2" y1="14.35" x2="46.70714375" y2="19.85714375" width="0.762" layer="16"/>
-<wire x1="42.6" y1="2.583334375" x2="42.6" y2="14.3" width="0.762" layer="16"/>
+<wire x1="42.6" y1="14.3" x2="42.6" y2="2.583334375" width="0.762" layer="16"/>
 <wire x1="46.70714375" y1="19.85714375" x2="46.78" y2="20.1" width="0.762" layer="16"/>
 <wire x1="42.6" y1="2.583334375" x2="42.26" y2="2.3" width="0.762" layer="16"/>
@@
 <wire x1="62.25" y1="26.5" x2="64.25" y2="24.5" width="0.762" layer="16"/>
 <wire x1="56.5" y1="26.5" x2="62.25" y2="26.5" width="0.762" layer="16"/>
-<wire x1="50.25" y1="20.25" x2="56.5" y2="26.5" width="0.762" layer="16"/>
+<wire x1="50.25" y1="20.25" x2="52.8" y2="22.8" width="0.762" layer="16"/>
+<wire x1="52.8" y1="22.8" x2="56.5" y2="26.5" width="0.762" layer="16"/>
 <wire x1="47" y1="20.25" x2="50.25" y2="20.25" width="0.762" layer="16"/>
 <wire x1="62.75" y1="11.75" x2="62.6" y2="11.54" width="0.762" layer="16"/>
 <wire x1="47" y1="20.25" x2="46.78" y2="20.1" width="0.762" layer="16"/>
-<wire x1="36.4" y1="14.3" x2="33.08" y2="10.98" width="0.762" layer="16"/>
-<wire x1="42.6" y1="14.3" x2="36.4" y2="14.3" width="0.762" layer="16"/>
 <via x="16" y="8" extent="1-16" drill="0.5"/>
 <via x="10" y="8" extent="1-16" drill="0.5"/>
@@
 <vertex x="70.1" y="29.8"/>
 </polygon>
-<wire x1="33.08" y1="10.98" x2="33.08" y2="9" width="0.762" layer="16"/>
 <wire x1="21.8" y1="11.9" x2="23" y2="13.1" width="0.762" layer="16"/>
-<wire x1="19.9" y1="11.9" x2="21.8" y2="11.9" width="0.762" layer="16"/>
+<wire x1="21.8" y1="11.9" x2="19.9" y2="11.9" width="0.762" layer="16"/>
+<wire x1="19.9" y1="11.9" x2="16" y2="8" width="0.762" layer="16"/>
+<wire x1="23" y1="13.1" x2="27.5" y2="17.6" width="0.762" layer="16"/>
+<wire x1="37.5" y1="17.6" x2="45.5" y2="25.6" width="0.762" layer="16"/>
+<wire x1="45.5" y1="25.6" x2="50" y2="25.6" width="0.762" layer="16"/>
+<wire x1="50" y1="25.6" x2="52.8" y2="22.8" width="0.762" layer="16"/>
+<wire x1="27.5" y1="17.6" x2="37.5" y2="17.6" width="0.762" layer="16"/>
+<wire x1="33.08" y1="9" x2="38.38" y2="14.3" width="0.762" layer="16"/>
+<wire x1="38.38" y1="14.3" x2="41.25" y2="14.3" width="0.762" layer="16"/>
+<wire x1="41.3" y1="14.3" x2="42.6" y2="14.3" width="0.762" layer="16"/>
+<wire x1="41.3" y1="14.3" x2="41.25" y2="14.3" width="0.762" layer="16"/>
+<wire x1="41.25" y1="14.3" x2="41.2" y2="14.35" width="0.762" layer="16"/>
 </signal>
 <signal name="+5V" class="1">
